File: diamond-mine-shimmer.kicad_sch (KiCad schematic)
At the start: 16 parts, among them Q1 2N3904, Q2 2N3906, Q3 2N3906, U1 CD4093BE

Commit message: x
Connections:
- net DARK: no longer U1.3 (1Y)
Other:
- note added: "SECTION G: LED DRIVERS Q1 (2N3904 NPN): FADE→10k→base, Steady LEDs VDD→1.5k→LED→Q1col Q2 (2N3906 PNP): OSC1→100k→base, Twinkle1 VDD→Q2emit→Q2col→LED→2.2k→GND Q3 (2N3906 PNP): OSC2→100k→base, Twinkle2 VDD→Q3emit→Q3col→LED→2.2k→GND"
- note removed: "SECTION G: LED DRIVERS Q1 (2N3904 NPN): FADE→10k→base, Steady LEDs VDD→1.5k→LED→Q1col Q2 (2N3906 PNP): OSC1→220k→base, Twinkle1 VDD→Q2emit→Q2col→LED→2.2k→GND Q3 (2N3906 PNP): OSC2→220k→base, Twinkle2 VDD→Q3emit→Q3col→LED→2.2k→GND"
- moved on the sheet: BT1, C_bypass, C_fade, D1, LDR1, Q1, Q2, Q3, RV1, R_charge, R_div1, R_div2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
